File: Qt_Py_J-Link/hardware/Qt_Py_j-link.brd (EAGLE design)
At the start: 38.1 x 44.2 mm, 13 parts, among them U1 Qt Py SAMD21

Commit message: reworked QT Py holes
Parts:
- removed U1: Qt Py SAMD21, home:QT_PY_TH
- added U2: QT Py SAMD21, home:QT_PY-SWD-TH
Connections:
- net !RESET: now also U2.!RESET; no longer U1.RESET
- net 3V3: now also U2.3V3@1, U2.3V3@2; no longer U1.3V3, U1.3V3@1
- net 5V: now also U2.5V@1, U2.5V@2; no longer U1.5V, U1.5V@1
- net A0: now also U2.A0@1, U2.A0@2; no longer U1.A0, U1.A0@1
- net GND: now also U2.GND@1, U2.GND@2; no longer U1.GND, U1.GND@1
- net N$1: now also U2.RX@1, U2.RX@2; no longer U1.RX, U1.RX@1
- net N$14: now also U2.TX@1, U2.TX@2; no longer U1.TX, U1.TX@1
- net N$2: now also U2.SCLK@1, U2.SCLK@2; no longer U1.SCLK, U1.SCLK@1
- net N$3: now also U2.MISO@1, U2.MISO@2; no longer U1.MISO, U1.MISO@1
- net N$4: now also U2.MOSI@1, U2.MOSI@2; no longer U1.MOSI, U1.MOSI@1
- net N$5: now also U2.A3@1, U2.A3@2; no longer U1.A3, U1.A3@1
- net N$6: now also U2.A1@1, U2.A1@2; no longer U1.A1, U1.A1@1
- net N$8: now also U2.A2@1, U2.A2@2; no longer U1.A2, U1.A2@1
- net SCL: now also U2.SCL@1, U2.SCL@2; no longer U1.SCL, U1.SCL@1
- net SDA: now also U2.SDA@1, U2.SDA@2; no longer U1.SDA, U1.SDA@1
- net SWCLK: now also U2.SWCLK; no longer U1.SWCLK
- net SWDIO: now also U2.SWDIO; no longer U1.SWDIO
Routing:
- net 3V3: track 45.6 -> 55.0 mm
- net GND: track 40.8 -> 47.0 mm
- net VT-TX: track 18.2 -> 17.1 mm
Other:
- board text added: "Access to SWDebug pads"
- board text added: "QT Py w/ J-Link"
- board text added: "Rev 1b"
- board text removed: "Qt Py w/ J-Link"
- board text removed: "access to swdebug pads"
